Commit message: Implement collision-aware UF850 pick-and-place workflow

File: ws/src/safe_servo_visualization/urdf/uf850_sensor_stack.urdf.xacro (robot description, xacro)
@@ -28,6 +28,7 @@
     </visual>
     <collision>
-      <origin xyz="0 0 0.0325" rpy="0 0 0"/>
-      <geometry><cylinder radius="0.045" length="0.065"/></geometry>
+      <!-- Avoid a false FCL contact at the rigid sensor/stand boundary. -->
+      <origin xyz="0 0 0.032" rpy="0 0 0"/>
+      <geometry><cylinder radius="0.045" length="0.064"/></geometry>
     </collision>
   </link>
